Commit message: Propagate the bluerobotics_models review fixes to the x500 packages
Assisted-by: Claude Fable 5 <noreply@anthropic.com>
Signed-off-by: Carlos Aguero <caguero@honurobotics.com>

File: x500_description/urdf/accessories.xacro (robot description, xacro)
@@ -10,9 +10,14 @@
 <robot xmlns:xacro="http://ros.org/wiki/xacro">
   <!-- ===== helpers ===== -->
+  <!-- Inertia tensors follow from the primitive geometry and the mass, so
+       they track the placeholder dimensions automatically. -->
   <xacro:macro name="_box_accessory" params="name xyz rpy parent size mass:=0.1">
+    <xacro:property name="d" value="${[float(v) for v in size.split()]}"/>
     <link name="${name}">
       <inertial>
         <mass value="${mass}"/>
-        <inertia ixx="0.0002" ixy="0" ixz="0" iyy="0.0002" iyz="0" izz="0.0002"/>
+        <inertia ixx="${float(mass)/12.0 * (d[1]**2 + d[2]**2)}" ixy="0" ixz="0"
+                 iyy="${float(mass)/12.0 * (d[0]**2 + d[2]**2)}" iyz="0"
+                 izz="${float(mass)/12.0 * (d[0]**2 + d[1]**2)}"/>
       </inertial>
       <visual>
@@ -47,6 +52,10 @@
     <link name="${name}">
       <inertial>
+        <origin xyz="0 0 0.06" rpy="0 0 0"/>
         <mass value="0.05"/>
-        <inertia ixx="0.0002" ixy="0" ixz="0" iyy="0.0002" iyz="0" izz="0.0002"/>
+        <!-- Slender mast (r 5 mm, l 0.12 m) about its centre; puck negligible. -->
+        <inertia ixx="${0.05/12.0 * (3*0.005**2 + 0.12**2)}" ixy="0" ixz="0"
+                 iyy="${0.05/12.0 * (3*0.005**2 + 0.12**2)}" iyz="0"
+                 izz="${0.05/2.0 * 0.005**2}"/>
       </inertial>
       <visual>
@@ -66,13 +75,12 @@
     </joint>
   </xacro:macro>
-  <!-- ===== recursive dispatcher: mount each config accessory by type ===== -->
+  <!-- ===== recursive dispatcher: mount each config accessory by type =====
+       The config `type` IS the macro name, invoked directly; an unknown type
+       fails the build loudly instead of silently mounting nothing. -->
   <xacro:macro name="mount_accessories" params="items parent:=base_link">
     <xacro:if value="${len(items) > 0}">
       <xacro:property name="a" value="${items[0]}"/>
-      <xacro:property name="t" value="${a['type']}"/>
-      <xacro:if value="${t == 'battery'}">           <xacro:battery            name="${a['name']}" xyz="${a['xyz']}" rpy="${a['rpy']}" parent="${parent}"/></xacro:if>
-      <xacro:if value="${t == 'companion_computer'}"><xacro:companion_computer name="${a['name']}" xyz="${a['xyz']}" rpy="${a['rpy']}" parent="${parent}"/></xacro:if>
-      <xacro:if value="${t == 'gimbal'}">            <xacro:gimbal             name="${a['name']}" xyz="${a['xyz']}" rpy="${a['rpy']}" parent="${parent}"/></xacro:if>
-      <xacro:if value="${t == 'gps_mast'}">          <xacro:gps_mast           name="${a['name']}" xyz="${a['xyz']}" rpy="${a['rpy']}" parent="${parent}"/></xacro:if>
+      <xacro:call macro="${a['type']}" name="${a['name']}"
+                  xyz="${a['xyz']}" rpy="${a['rpy']}" parent="${parent}"/>
       <xacro:mount_accessories items="${items[1:]}" parent="${parent}"/>
     </xacro:if>

File: x500_gazebo/model.sdf.xacro (robot description, xacro)
@@ -50,8 +50,8 @@
       <pose relative_to="base_link">0 0 0 0 0 0</pose>
       <inertial>
-        <mass>0.001</mass>
+        <mass>1e-5</mass>
         <inertia>
-          <ixx>1e-6</ixx><ixy>0</ixy><ixz>0</ixz>
-          <iyy>1e-6</iyy><iyz>0</iyz><izz>1e-6</izz>
+          <ixx>1e-8</ixx><ixy>0</ixy><ixz>0</ixz>
+          <iyy>1e-8</iyy><iyz>0</iyz><izz>1e-8</izz>
         </inertia>
       </inertial>
