Commit message: Name each X500 instance once and put its topics and frames under it
Signed-off-by: Carlos Agüero <caguero@honurobotics.com>
Assisted-by: Claude Fable 5.1 <noreply@anthropic.com>

File: x500_gazebo/model.sdf.xacro (robot description, xacro)
@@ -23,6 +23,9 @@
   <!-- Topic namespace: every part topic is /<topic_namespace>/<part name>/...
        on both sides (a GPS part's /fix). Per part, `gz_topic` / `topic`
-       override the gz side base; the bridge config is generated from the
-       same yaml, so gz and ROS sides stay in sync. -->
+       override the gz side base, under the namespace unless they start with
+       a slash; the bridge config is generated from the same yaml, so gz and
+       ROS sides stay in sync. The namespace is also the instance name: the
+       model name and, in a simulation, the prefix of every TF frame, so the
+       sensors' frame ids carry it. -->
   <xacro:property name="topic_ns" value="${cfg.get('topic_namespace', 'x500')}"/>
   <!-- The root link the assembly names (the config's base.name). -->
@@ -93,6 +96,7 @@
       <sensor name="${name}" type="navsat">
         <!-- Pin frame_id to the part's antenna frame: a URDF link, so TF
-             carries it. -->
-        <frame_id>${frame}</frame_id>
+             carries it, under the instance name, which is the prefix
+             robot_state_publisher puts on every frame of this instance. -->
+        <frame_id>${topic_ns}/${frame}</frame_id>
         <topic>${topic_base}/fix</topic>
         <always_on>1</always_on>
@@ -109,6 +113,7 @@
   <xacro:macro name="gz_part" params="ptype name parent xyz rpy collision joint axis info">
     <xacro:part_entry name="${name}"/>
+    <xacro:property name="topic_override" value="${entry.get('gz_topic', entry.get('topic', name))}"/>
     <xacro:property name="topic_base"
-                    value="${entry.get('gz_topic', entry.get('topic', topic_ns + '/' + name))}"/>
+                    value="${topic_override if topic_override.startswith('/') else topic_ns + '/' + topic_override}"/>
     <!-- A propeller on a fixed joint (a spare, say) is lumped away and
          drives nothing. -->
@@ -122,10 +127,13 @@
   <xacro:macro name="gz_no_slot" params="name parent xyz rpy:='0 0 0'">
   </xacro:macro>
-  <model name="x500">
+  <!-- Named after the instance (the config's topic_namespace, or the name
+       option of configure_vehicle.py): the model name, the topic namespace
+       and, in the launch, the TF prefix are one and the same. -->
+  <model name="${topic_ns}">
     <include merge="true">
       <uri>$(arg urdf_uri)</uri>
     </include>
     <!-- Joint states for the rotor joints, so robot_state_publisher can
-         animate the props in RViz. Bridged to /joint_states. -->
+         animate the props in RViz. Bridged to /<ns>/joint_states. -->
     <plugin filename="gz-sim-joint-state-publisher-system"
             name="gz::sim::systems::JointStatePublisher">
@@ -146,5 +154,5 @@
       </inertial>
       <sensor name="imu" type="imu">
-        <frame_id>${base_name}</frame_id>
+        <frame_id>${topic_ns}/${base_name}</frame_id>
         <topic>${topic_ns}/imu</topic>
         <always_on>1</always_on>
@@ -164,5 +172,5 @@
       </sensor>
       <sensor name="air_pressure" type="air_pressure">
-        <frame_id>${base_name}</frame_id>
+        <frame_id>${topic_ns}/${base_name}</frame_id>
         <topic>${topic_ns}/air_pressure</topic>
         <always_on>1</always_on>
@@ -173,5 +181,5 @@
       </sensor>
       <sensor name="magnetometer" type="magnetometer">
-        <frame_id>${base_name}</frame_id>
+        <frame_id>${topic_ns}/${base_name}</frame_id>
         <topic>${topic_ns}/mag</topic>
         <always_on>1</always_on>
