Commit message: Replace the X500 placeholder meshes with glTF parts modeled from dimensions
Assisted-by: Claude Code (claude-opus-5-5)
Co-Authored-By: Claude Opus 5.5 <noreply@anthropic.com>
Signed-off-by: Carlos Agüero <caguero@honurobotics.com>

File: holybro_parts/urdf/battery_4s.urdf.xacro (robot description, xacro)
@@ -2,7 +2,10 @@
 <!--
   battery_4s part macro: a 4S LiPo pack, the largest movable mass and biggest CG lever.
-  Sized primitive placeholder (dims from product pages); swap for a real
-  mesh when delivered. Mass and pose matter: accessories set the vehicle
-  center of gravity.
+  Visual: models/battery_4s/battery_4s_visual.glb, a 145 x 48 x 38 mm pack
+  with its leads, XT60 and balance plugs. Its datum, the part frame, is the
+  center of the pack's top face, which straps against the battery pad; the
+  pack hangs below it, so the inertia and the collision box sit half its
+  height down. Mass and pose matter: accessories set the vehicle center of
+  gravity.
   Contract (see parts.xacro): <part>_info exports the metadata (attach,
   slots, frames, drive); <part> instantiates the link, its mounting joint
@@ -25,4 +28,5 @@
     <link name="${name}">
       <inertial>
+        <origin xyz="0 0 ${-_d[2]/2}" rpy="0 0 0"/>
         <mass value="${_m}"/>
         <inertia ixx="${_m/12.0 * (_d[1]**2 + _d[2]**2)}" ixy="0" ixz="0"
@@ -30,10 +34,8 @@
                  izz="${_m/12.0 * (_d[0]**2 + _d[1]**2)}"/>
       </inertial>
-      <visual>
-        <geometry><box size="${_d[0]} ${_d[1]} ${_d[2]}"/></geometry>
-        <material name="${name}_mat"><color rgba="0.2 0.2 0.22 1"/></material>
-      </visual>
+      <xacro:part_visual mesh="package://holybro_parts/models/battery_4s/battery_4s_visual.glb"/>
       <xacro:if value="${collision}">
         <collision>
+          <origin xyz="0 0 ${-_d[2]/2}" rpy="0 0 0"/>
           <geometry><box size="${_d[0]} ${_d[1]} ${_d[2]}"/></geometry>
         </collision>

File: holybro_parts/urdf/companion_computer.urdf.xacro (robot description, xacro)
@@ -2,6 +2,9 @@
 <!--
   companion_computer part macro: a companion computer (RPi 4 / Jetson class) on the payload plate.
-  Sized primitive placeholder (dims from product pages); swap for a real
-  mesh when delivered. Mass and pose matter: accessories set the vehicle
+  Visual: models/companion_computer/companion_computer_visual.glb, a
+  Raspberry Pi 5 on 6 mm standoffs, its ports toward the rear. Its datum, the
+  part frame, is the center of the 58 x 49 mm hole pattern on the standoffs'
+  lower faces; the board sits above it, so the inertia and the collision box
+  sit above the datum. Mass and pose matter: accessories set the vehicle
   center of gravity.
   Contract (see parts.xacro): <part>_info exports the metadata (attach,
@@ -25,4 +28,5 @@
     <link name="${name}">
       <inertial>
+        <origin xyz="0 0 ${_d[2]/2}" rpy="0 0 0"/>
         <mass value="${_m}"/>
         <inertia ixx="${_m/12.0 * (_d[1]**2 + _d[2]**2)}" ixy="0" ixz="0"
@@ -30,11 +34,10 @@
                  izz="${_m/12.0 * (_d[0]**2 + _d[1]**2)}"/>
       </inertial>
-      <visual>
-        <geometry><box size="${_d[0]} ${_d[1]} ${_d[2]}"/></geometry>
-        <material name="${name}_mat"><color rgba="0.2 0.2 0.22 1"/></material>
-      </visual>
+      <xacro:part_visual mesh="package://holybro_parts/models/companion_computer/companion_computer_visual.glb"/>
       <xacro:if value="${collision}">
         <collision>
-          <geometry><box size="${_d[0]} ${_d[1]} ${_d[2]}"/></geometry>
+          <!-- The visual's extent: board, cooler and the ports reaching back. -->
+          <origin xyz="-0.01125 0 0.0116" rpy="0 0 0"/>
+          <geometry><box size="0.0875 0.057 0.0232"/></geometry>
         </collision>
       </xacro:if>

File: holybro_parts/urdf/gimbal_camera.urdf.xacro (robot description, xacro)
@@ -2,7 +2,9 @@
 <!--
   gimbal_camera part macro: a gimbal payload camera (A8 mini class) slung below and forward.
-  Sized primitive placeholder (dims from product pages); swap for a real
-  mesh when delivered. Mass and pose matter: accessories set the vehicle
-  center of gravity.
+  Visual: models/gimbal_camera/gimbal_camera_visual.glb, a SIYI A8 mini
+  (55 x 55 x 70 mm). Its datum, the part frame, is the center of the mounting
+  plate's upper face, which bolts under the payload rails; the gimbal hangs
+  below it, so the inertia and the collision box sit half its height down.
+  Mass and pose matter: accessories set the vehicle center of gravity.
   Contract (see parts.xacro): <part>_info exports the metadata (attach,
   slots, frames, drive); <part> instantiates the link, its mounting joint
@@ -25,4 +27,5 @@
     <link name="${name}">
       <inertial>
+        <origin xyz="0 0 ${-_d[2]/2}" rpy="0 0 0"/>
         <mass value="${_m}"/>
         <inertia ixx="${_m/12.0 * (_d[1]**2 + _d[2]**2)}" ixy="0" ixz="0"
@@ -30,11 +33,10 @@
                  izz="${_m/12.0 * (_d[0]**2 + _d[1]**2)}"/>
       </inertial>
-      <visual>
-        <geometry><box size="${_d[0]} ${_d[1]} ${_d[2]}"/></geometry>
-        <material name="${name}_mat"><color rgba="0.2 0.2 0.22 1"/></material>
-      </visual>
+      <xacro:part_visual mesh="package://holybro_parts/models/gimbal_camera/gimbal_camera_visual.glb"/>
       <xacro:if value="${collision}">
         <collision>
-          <geometry><box size="${_d[0]} ${_d[1]} ${_d[2]}"/></geometry>
+          <!-- The visual's extent, mounting plate to the bottom of the head. -->
+          <origin xyz="0 0 -0.0345" rpy="0 0 0"/>
+          <geometry><box size="0.055 0.055 0.069"/></geometry>
         </collision>
       </xacro:if>

File: holybro_parts/urdf/gps_mast.urdf.xacro (robot description, xacro)
@@ -2,7 +2,10 @@
 <!--
   gps_mast part macro: a GPS/RTK module on a mast: thin mast plus puck on top. One parametric mount covers the M8N to M10 to F9P family (retune mass/height per module).
-  Sized primitive placeholder (dims from product pages); swap for a real
-  mesh when delivered. Mass and pose matter: accessories set the vehicle
-  center of gravity.
+  Visual: models/gps_mast/gps_mast_visual.glb, a folding GPS mast modeled
+  from the kit's measured sizes with an M10 puck (50 mm, 14.4 mm tall) on its
+  tray. Its datum, the part frame, is the center of the base clamp's lower
+  face on the mast axis, where it sits on the payload platform; the puck's
+  lid is 0.147 m up.
+  Mass and pose matter: accessories set the vehicle center of gravity.
   Contract (see parts.xacro): <part>_info exports the metadata (attach,
   slots, frames, drive); <part> instantiates the link, its mounting joint
@@ -18,5 +21,5 @@
         ),
         frames=dict(
-            antenna=dict(xyz='0 0 0.13', rpy='0 0 0'),
+            antenna=dict(xyz='0 0 0.142', rpy='0 0 0'),
         ))}"/>
   </xacro:macro>
@@ -26,21 +29,29 @@
     <link name="${name}">
       <inertial>
-        <origin xyz="0 0 0.06" rpy="0 0 0"/>
+        <!-- 32 g puck at 0.14 m over an 18 g mount spread up the mast: the
+             center of mass is about 0.10 m up. Treated as a slender rod of
+             the mount's height about that point, puck included. -->
+        <origin xyz="0 0 0.10" rpy="0 0 0"/>
         <mass value="0.05"/>
-        <!-- Slender mast (r 5 mm, l 0.12 m) about its centre; puck negligible. -->
-        <inertia ixx="${0.05/12.0 * (3*0.005**2 + 0.12**2)}" ixy="0" ixz="0"
-                 iyy="${0.05/12.0 * (3*0.005**2 + 0.12**2)}" iyz="0"
-                 izz="${0.05/2.0 * 0.005**2}"/>
+        <inertia ixx="${0.05/12.0 * (3*0.005**2 + 0.147**2)}" ixy="0" ixz="0"
+                 iyy="${0.05/12.0 * (3*0.005**2 + 0.147**2)}" iyz="0"
+                 izz="${0.032/2.0 * 0.025**2}"/>
       </inertial>
-      <visual>
-        <origin xyz="0 0 0.06" rpy="0 0 0"/>
-        <geometry><cylinder radius="0.005" length="0.12"/></geometry>
-        <material name="${name}_mast"><color rgba="0.15 0.15 0.15 1"/></material>
-      </visual>
-      <visual>
-        <origin xyz="0 0 0.13" rpy="0 0 0"/>
-        <geometry><cylinder radius="0.028" length="0.018"/></geometry>
-        <material name="${name}_puck"><color rgba="0.85 0.85 0.85 1"/></material>
-      </visual>
+      <xacro:part_visual mesh="package://holybro_parts/models/gps_mast/gps_mast_visual.glb"/>
+      <xacro:if value="${collision}">
+        <!-- Base clamp, mast and puck, as cylinders on the mast axis. -->
+        <collision name="clamp">
+          <origin xyz="0 0 0.0057" rpy="0 0 0"/>
+          <geometry><cylinder radius="0.015" length="0.0186"/></geometry>
+        </collision>
+        <collision name="mast">
+          <origin xyz="0 0 0.0705" rpy="0 0 0"/>
+          <geometry><cylinder radius="0.0046" length="0.111"/></geometry>
+        </collision>
+        <collision name="puck">
+          <origin xyz="0 0 0.1373" rpy="0 0 0"/>
+          <geometry><cylinder radius="0.026" length="0.023"/></geometry>
+        </collision>
+      </xacro:if>
     </link>
     <xacro:part_joint name="${name}" parent="${parent}" xyz="${xyz}" rpy="${rpy}"

File: holybro_parts/urdf/parts.xacro (robot description, xacro)
@@ -55,15 +55,22 @@
 <robot xmlns:xacro="http://ros.org/wiki/xacro">
   <!-- ===== helpers used by every part macro ===== -->
-  <!-- glTF meshes are Y-up by specification and the delivered .glb files
-       conform. RViz and other ROS tools rotate them to Z-up on load; Gazebo
-       does not (it shows the data as is), so the URDF Gazebo merges is
-       expanded with gltf_up:=z, which pre-rotates every glTF visual by +90
-       degrees about x. The installed ROS URDF keeps gltf_up=y (no rotation). -->
+  <!-- Delivered .glb parts are in glTF's own axes (Honu glTF Asset Profile,
+       Axes): +Y up, +Z forward, origin on the part's datum. Placing one on a
+       link takes a fixed rotation, roll 90 degrees then yaw 90 degrees, and
+       the consumers differ in how much of it they apply themselves:
+         RViz (Lyrical and later) rolls glTF +90 about x on load, so the ROS
+           URDF carries only the yaw: rpy 0 0 1.5708 (gltf_up:=y, the default);
+         Gazebo applies nothing, so the URDF Gazebo merges carries the whole
+           rotation: rpy 1.5708 0 1.5708 (x500_gazebo expands with gltf_up:=z).
+       A part may add a yaw about the link's z axis on top, e.g. to clock a
+       motor's mounting pattern. -->
   <xacro:arg name="gltf_up" default="y"/>
-  <xacro:property name="gltf_visual_rpy" value="${'1.5708 0 0' if '$(arg gltf_up)' == 'z' else '0 0 0'}"/>
-  <!-- A part's visual mesh, with the glTF up axis handling above. -->
-  <xacro:macro name="part_visual" params="mesh xyz:='0 0 0'">
+  <xacro:property name="gltf_roll" value="${1.5708 if '$(arg gltf_up)' == 'z' else 0.0}"/>
+  <!-- A part's visual: one .glb, placed at xyz with the rotation above. No
+       <material>: the file's own PBR materials render, and a URDF or SDF
+       material would replace every one of them. -->
+  <xacro:macro name="part_visual" params="mesh xyz:='0 0 0' yaw:=0">
     <visual>
-      <origin xyz="${xyz}" rpy="${gltf_visual_rpy}"/>
+      <origin xyz="${xyz}" rpy="${gltf_roll} 0 ${1.5708 + float(yaw)}"/>
       <geometry>
         <mesh filename="${mesh}"/>
@@ -131,6 +138,6 @@
   <xacro:include filename="$(find holybro_parts)/urdf/gimbal_camera.urdf.xacro"/>
   <xacro:include filename="$(find holybro_parts)/urdf/gps_mast.urdf.xacro"/>
-  <xacro:include filename="$(find holybro_parts)/urdf/prop_1345_ccw.urdf.xacro"/>
-  <xacro:include filename="$(find holybro_parts)/urdf/prop_1345_cw.urdf.xacro"/>
+  <xacro:include filename="$(find holybro_parts)/urdf/prop_1045_ccw.urdf.xacro"/>
+  <xacro:include filename="$(find holybro_parts)/urdf/prop_1045_cw.urdf.xacro"/>
   <xacro:include filename="$(find holybro_parts)/urdf/x500_airframe.urdf.xacro"/>
 </robot>

File: holybro_parts/urdf/prop_1045_ccw.urdf.xacro (robot description, xacro)
@@ -1,11 +1,14 @@
 <?xml version="1.0"?>
 <!--
-  prop_1345_ccw part macro: a 1345 propeller with its rotating motor bell,
-  the counter clockwise rotor of the X500 quad X pair.
-  Mesh, inertia and collision are PX4's BSD 3 Clause x500 values
-  (models/LICENSE); the bell is the HoverGames 5010, a placeholder for the
-  Holybro 2216. Drive: the multicopter motor plant constants a simulator
-  needs to spin this prop on its joint (PX4's values; identify for the
-  real 2216 + 1045 pair).
+  prop_1045_ccw part macro: a 1045 (10 x 4.5 inch) propeller with the
+  rotating bell of its Holybro 2216 motor, the counter clockwise rotor of the X500
+  quad X pair.
+  Visuals: models/prop_1045_ccw/prop_1045_ccw_visual.glb and
+  models/motor_2216/motor_2216_bell_visual.glb. Both datums are the prop
+  seat on the rotation axis (the bell's top face, the hub's lower face),
+  which is this part's frame; the airframe places the rotor slot there.
+  Inertia, collision thickness and the drive constants are still PX4's
+  BSD 3 Clause x500 values (models/LICENSE); identify them for the real
+  2216 + 1045 pair.
   Contract (see parts.xacro): <part>_info exports the metadata (attach,
   slots, frames, drive); <part> instantiates the link, its mounting joint
@@ -13,5 +16,5 @@
 -->
 <robot xmlns:xacro="http://ros.org/wiki/xacro">
-  <xacro:macro name="prop_1345_ccw_info">
+  <xacro:macro name="prop_1045_ccw_info">
     <xacro:property name="part_info" scope="parent" value="${dict(
         attach='0 0 0',
@@ -25,31 +28,21 @@
                    velocity_slowdown_sim=10))}"/>
   </xacro:macro>
-  <xacro:macro name="prop_1345_ccw"
+  <xacro:macro name="prop_1045_ccw"
                params="name parent xyz:='0 0 0' rpy:='0 0 0' collision:=true joint:=fixed axis:='0 0 1'">
-    <xacro:prop_1345_ccw_info/>
+    <xacro:prop_1045_ccw_info/>
     <link name="${name}">
       <inertial>
         <mass value="0.016076923076923075"/>
-        <inertia ixx="3.8464910483993325e-07" ixy="0" ixz="0"
-                 iyy="2.6115851691700804e-05" iyz="0" izz="2.649858234714004e-05"/>
+        <inertia ixx="2.6115851691700804e-05" ixy="0" ixz="0"
+                 iyy="3.8464910483993325e-07" iyz="0" izz="2.649858234714004e-05"/>
       </inertial>
-      <visual>
-        <origin xyz="-0.022 -0.14638461538461536 -0.016" rpy="0 0 0"/>
-        <geometry>
-          <mesh filename="package://holybro_parts/models/prop_1345_ccw/1345_prop_ccw.stl"
-                scale="0.8461538461538461 0.8461538461538461 0.8461538461538461"/>
-        </geometry>
-        <material name="${name}_grey"><color rgba="0.25 0.25 0.25 1"/></material>
-      </visual>
-      <visual>
-        <origin xyz="0 0 -0.032" rpy="0 0 0"/>
-        <geometry>
-          <mesh filename="package://holybro_parts/models/prop_1345_ccw/5010Bell.dae"/>
-        </geometry>
-      </visual>
+      <xacro:part_visual mesh="package://holybro_parts/models/motor_2216/motor_2216_bell_visual.glb"/>
+      <xacro:part_visual mesh="package://holybro_parts/models/prop_1045_ccw/prop_1045_ccw_visual.glb"/>
       <xacro:if value="${collision}">
         <collision>
+          <!-- The blade's span at hub height, along the part's Y like the visual. -->
+          <origin xyz="0 0 0.006" rpy="0 0 0"/>
           <geometry>
-            <box size="0.2792307692307692 0.016923076923076923 0.0008461538461538462"/>
+            <box size="0.016923076923076923 0.254 0.0008461538461538462"/>
           </geometry>
         </collision>

File: holybro_parts/urdf/prop_1045_cw.urdf.xacro (robot description, xacro)
@@ -1,11 +1,14 @@
 <?xml version="1.0"?>
 <!--
-  prop_1345_cw part macro: a 1345 propeller with its rotating motor bell,
-  the clockwise rotor of the X500 quad X pair.
-  Mesh, inertia and collision are PX4's BSD 3 Clause x500 values
-  (models/LICENSE); the bell is the HoverGames 5010, a placeholder for the
-  Holybro 2216. Drive: the multicopter motor plant constants a simulator
-  needs to spin this prop on its joint (PX4's values; identify for the
-  real 2216 + 1045 pair).
+  prop_1045_cw part macro: a 1045 (10 x 4.5 inch) propeller with the
+  rotating bell of its Holybro 2216 motor, the clockwise rotor of the X500
+  quad X pair.
+  Visuals: models/prop_1045_cw/prop_1045_cw_visual.glb and
+  models/motor_2216/motor_2216_bell_visual.glb. Both datums are the prop
+  seat on the rotation axis (the bell's top face, the hub's lower face),
+  which is this part's frame; the airframe places the rotor slot there.
+  Inertia, collision thickness and the drive constants are still PX4's
+  BSD 3 Clause x500 values (models/LICENSE); identify them for the real
+  2216 + 1045 pair.
   Contract (see parts.xacro): <part>_info exports the metadata (attach,
   slots, frames, drive); <part> instantiates the link, its mounting joint
@@ -13,5 +16,5 @@
 -->
 <robot xmlns:xacro="http://ros.org/wiki/xacro">
-  <xacro:macro name="prop_1345_cw_info">
+  <xacro:macro name="prop_1045_cw_info">
     <xacro:property name="part_info" scope="parent" value="${dict(
         attach='0 0 0',
@@ -25,31 +28,21 @@
                    velocity_slowdown_sim=10))}"/>
   </xacro:macro>
-  <xacro:macro name="prop_1345_cw"
+  <xacro:macro name="prop_1045_cw"
                params="name parent xyz:='0 0 0' rpy:='0 0 0' collision:=true joint:=fixed axis:='0 0 1'">
-    <xacro:prop_1345_cw_info/>
+    <xacro:prop_1045_cw_info/>
     <link name="${name}">
       <inertial>
         <mass value="0.016076923076923075"/>
-        <inertia ixx="3.8464910483993325e-07" ixy="0" ixz="0"
-                 iyy="2.6115851691700804e-05" iyz="0" izz="2.649858234714004e-05"/>
+        <inertia ixx="2.6115851691700804e-05" ixy="0" ixz="0"
+                 iyy="3.8464910483993325e-07" iyz="0" izz="2.649858234714004e-05"/>
       </inertial>
-      <visual>
-        <origin xyz="-0.022 -0.14638461538461536 -0.016" rpy="0 0 0"/>
-        <geometry>
-          <mesh filename="package://holybro_parts/models/prop_1345_cw/1345_prop_cw.stl"
-                scale="0.8461538461538461 0.8461538461538461 0.8461538461538461"/>
-        </geometry>
-        <material name="${name}_grey"><color rgba="0.25 0.25 0.25 1"/></material>
-      </visual>
-      <visual>
-        <origin xyz="0 0 -0.032" rpy="0 0 0"/>
-        <geometry>
-          <mesh filename="package://holybro_parts/models/prop_1345_cw/5010Bell.dae"/>
-        </geometry>
-      </visual>
+      <xacro:part_visual mesh="package://holybro_parts/models/motor_2216/motor_2216_bell_visual.glb"/>
+      <xacro:part_visual mesh="package://holybro_parts/models/prop_1045_cw/prop_1045_cw_visual.glb"/>
       <xacro:if value="${collision}">
         <collision>
+          <!-- The blade's span at hub height, along the part's Y like the visual. -->
+          <origin xyz="0 0 0.006" rpy="0 0 0"/>
           <geometry>
-            <box size="0.2792307692307692 0.016923076923076923 0.0008461538461538462"/>
+            <box size="0.016923076923076923 0.254 0.0008461538461538462"/>
           </geometry>
         </collision>
